File: TouchKey/IambicKey.sch (EAGLE design)
At the start: 12 parts, among them Q1 MOSFET-NCHANNELSMD, Q2 MOSFET-NCHANNELSMD, U1 AT42QT1012, U2 AT42QT1012

Commit message: Replaced most through hole components with SMD equivilents
Parts:
- added TP1, TP2, TP3, TP4, TP5: TPTP20SQ, testpad:TPTP20SQ
Connections:
- new net N$10: Q1.D, TP1.TP
- new net N$11: Q2.D, TP2.TP
- net GND: now also TP4.TP, TP5.TP
- net VCC: now also TP3.TP
Changed lines of the file:
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@@
 <part name="U$1" library="morseSounder" deviceset="PADDLE" device=""/>
 <part name="U$2" library="morseSounder" deviceset="PADDLE" device=""/>
+<part name="TP1" library="testpad" deviceset="TP" device="TP20SQ"/>
+<part name="TP2" library="testpad" deviceset="TP" device="TP20SQ"/>
+<part name="TP3" library="testpad" deviceset="TP" device="TP20SQ"/>
+<part name="TP4" library="testpad" deviceset="TP" device="TP20SQ"/>
+<part name="P+7" library="SparkFun" deviceset="VCC" device=""/>
+<part name="GND7" library="SparkFun" deviceset="GND" device=""/>
+<part name="TP5" library="testpad" deviceset="TP" device="TP20SQ"/>
+<part name="GND8" library="SparkFun" deviceset="GND" device=""/>
 </parts>
 <sheets>
@@
 <instance part="U$1" gate="G$1" x="2.54" y="48.26" rot="R180"/>
 <instance part="U$2" gate="G$1" x="2.54" y="7.62" rot="R180"/>
+<instance part="TP1" gate="G$1" x="99.06" y="55.88"/>
+<instance part="TP2" gate="G$1" x="99.06" y="15.24"/>
+<instance part="TP3" gate="G$1" x="68.58" y="76.2"/>
+<instance part="TP4" gate="G$1" x="76.2" y="76.2"/>
+<instance part="P+7" gate="1" x="68.58" y="73.66" rot="R180"/>
+<instance part="GND7" gate="1" x="76.2" y="71.12"/>
+<instance part="TP5" gate="G$1" x="83.82" y="76.2"/>
+<instance part="GND8" gate="1" x="83.82" y="71.12"/>
 </instances>
 <busses>
@@
 <pinref part="GND6" gate="1" pin="GND"/>
 </segment>
+<segment>
+<pinref part="TP4" gate="G$1" pin="TP"/>
+<pinref part="GND7" gate="1" pin="GND"/>
+</segment>
+<segment>
+<pinref part="TP5" gate="G$1" pin="TP"/>
+<pinref part="GND8" gate="1" pin="GND"/>
+</segment>
 </net>
 <net name="N$1" class="0">
@@
 <pinref part="C1" gate="G$1" pin="1"/>
 <pinref part="P+6" gate="1" pin="VCC"/>
+</segment>
+<segment>
+<pinref part="TP3" gate="G$1" pin="TP"/>
+<pinref part="P+7" gate="1" pin="VCC"/>
 </segment>
 </net>
@@
 </segment>
 </net>
+<net name="N$10" class="0">
+<segment>
+<pinref part="Q1" gate="G$1" pin="D"/>
+<pinref part="TP1" gate="G$1" pin="TP"/>
+</segment>
+</net>
+<net name="N$11" class="0">
+<segment>
+<pinref part="Q2" gate="G$1" pin="D"/>
+<pinref part="TP2" gate="G$1" pin="TP"/>
+</segment>
+</net>
