File: PCB/morseSounder.sch (EAGLE design)
At the start: 77 parts, among them IC1 LM386M-1, IC5 LM321MF, J1 AVR_SPI_PRG_6PTH, J2 POWERPOLE_POWER25A_HORIZONTAL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, J3 POWER_JACKPTH, Q1 MMBT3904, Q2 MMBT3904, Q3 MMBT3904, T1 MMBTA42, U1 ATMEGA168

Commit message: * Removed the pair of unused opto-isolators. * Commenced tidying up the schematic. & Removal of 3rd opto-isolator may prove tricky...
Parts:
- removed OK2, OK3: 4N35, optocoupler:4N35
- R28, R29: value 750 -> 330
Connections:
- removed net AVR_DASH: U1.PC3(ADC3)
- removed net AVR_DOT: U1.PC2(ADC2)
- removed net AVR_KEY_DASH: OK3.COL
- removed net AVR_KEY_DOT: OK2.COL
- removed net N$34: LED2.C, OK3.A
- removed net N$35: LED3.C, OK2.A
- net +12V: now also C19.1, U$5.IN
- net GND: no longer OK2.EMI, OK3.EMI
- net KEY_DASH: now also LED3.C, U1.PC3(ADC3); no longer OK3.C
- net KEY_DOT: now also LED2.C, U1.PC2(ADC2); no longer OK2.C
- net VIN: no longer C19.1, U$5.IN
Other:
- note added: "Power Supplies"
- note removed: "AVR opto isolators"
- moved on the sheet: C19, C20, LED2, LED3, LED4, R1, R14, R15, R28, R29, R30, TP7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

Commit message: * Removed opto-isolator driving the amplifier. Swapped to a high side MOSFET driver.     Note this makes the micro mandatory. * Added input protection for the key.
Parts:
- removed JP1, JP3, JP4: JUMPER-3SMD, SparkFun:JUMPER-3SMD
- removed LED1: (no value), SparkFun:LED-3MM-NO_SILK
- removed OK1: 4N35, optocoupler:4N35
- removed R27: 750, SparkFun:RESISTOR0805-RES
- added D1, D2: 200mA/70V, SparkFun-DiscreteSemi:BAV99
- added D4: 0.5A/40V/420mV, SparkFun-DiscreteSemi:DIODE-SCHOTTKY-PMEG4005EJ
- added Q4: 2.5A/30V/105mΩ, SparkFun-DiscreteSemi:MOSFET_PCH-DMG2307L
- added Q5: MMBT3904, transistor:MMBT3904LT1-NPN-SOT23-BEC
- added R17, R18: 10k, SparkFun:RESISTOR0805-RES
- added TP9: TEST-POINT3X5, SparkFun-Connectors:TEST-POINT3X5
Connections:
- removed net KEY_INPUT: JP1.1, JP3.2
- removed net N$10: LED1.C, OK1.A
- removed net N$30: JP4.2, R27.2
- removed net N$31: JP1.2, OK1.C
- removed net N$32: LED1.A, R27.1
- new net N$16: Q5.B, R18.2
- new net N$17: Q4.G, Q5.C, R17.1
- new net N$4: D4.A, J2.V+
- net +12V: now also Q4.S, R17.2; no longer JP4.3, OK1.COL
- net AVR_KEY_OUT: now also R18.1, TP9.1; no longer JP4.1
- net AVR_VCC: now also D1.C2, D2.C2
- net GND: now also D1.A1, D2.A1, Q5.E; no longer JP1.3
- net KEY_DASH: now also D2.COM; no longer JP3.3
- net KEY_DOT: now also D1.COM; no longer JP3.1
- net KEY_IN: now also Q4.D; no longer OK1.EMI
- net VIN: now also D4.C; no longer J2.V+
Other:
- note removed: "for keyer"
- note removed: "for non keyer"
- note removed: "non keyer Input selection"
- moved on the sheet: C13, C14, C15, R14, R15, R24, TP7, U$3G$1
