File: PCB/morseSounder.sch (EAGLE design)
At the start: 81 parts, among them IC1 LM386M-1, IC5 LM321MF, J1 AVR_SPI_PRG_6PTH, J2 POWERPOLE_POWER25A_HORIZONTAL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, J3 POWER_JACKPTH, Q1 MMBT3904, Q2 MMBT3904, Q3 MMBT3904, Q4 2.5A/30V/105mΩ, Q5 MMBT3904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

Commit message: Added some decoupling capacitors and tidied silk screen
Parts:
- added C8: 100n, SparkFun:CAP0805
- added C9: 10n, SparkFun:CAP0805
- added U$7: LOGO_SUWSLOGO_LARGE, morseSounder:LOGO_SUWSLOGO_LARGE
Connections:
- net AVR_VCC: now also C8.2, C9.2
- net GND: now also C8.1, C9.1
Changed lines of the file:
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@@
 <part name="R22" library="SparkFun" deviceset="RESISTOR" device="0805-RES" value="15K"/>
 <part name="U1" library="SparkFun-IC-Microcontroller" deviceset="ATMEGA328P_TQFP" device="" value="ATMEGA328P_TQFP"/>
+<part name="U$7" library="morseSounder" deviceset="LOGO_SUWS" device="LOGO_LARGE"/>
+<part name="C8" library="SparkFun" deviceset="CAP" device="0805" value="100n"/>
+<part name="C9" library="SparkFun" deviceset="CAP" device="0805" value="10n"/>
+<part name="GND21" library="supply1" deviceset="GND" device=""/>
 </parts>
 <sheets>
@@
 <instance part="R22" gate="G$1" x="152.4" y="-12.7" rot="R90"/>
 <instance part="U1" gate="U$1" x="66.04" y="142.24"/>
+<instance part="U$7" gate="G$1" x="58.42" y="99.06"/>
+<instance part="C8" gate="G$1" x="116.84" y="160.02" rot="R180"/>
+<instance part="C9" gate="G$1" x="124.46" y="160.02" rot="R180"/>
+<instance part="GND21" gate="1" x="109.22" y="152.4"/>
 </instances>
 <busses>
@@
 <pinref part="U1" gate="U$1" pin="GND@5"/>
 <pinref part="U1" gate="U$1" pin="AGND"/>
+</segment>
+<segment>
+<pinref part="C9" gate="G$1" pin="1"/>
+<pinref part="C8" gate="G$1" pin="1"/>
+<wire x1="124.46" y1="154.94" x2="116.84" y2="154.94" width="0.1524" layer="91"/>
+<wire x1="116.84" y1="154.94" x2="109.22" y2="154.94" width="0.1524" layer="91"/>
+<pinref part="GND21" gate="1" pin="GND"/>
+<junction x="109.22" y="154.94"/>
 </segment>
 </net>
@@
 <junction x="142.24" y="-5.08"/>
 </segment>
-</net>
+<segment>
+<pinref part="C9" gate="G$1" pin="2"/>
+<pinref part="C8" gate="G$1" pin="2"/>
+<wire x1="124.46" y1="162.56" x2="116.84" y2="162.56" width="0.1524" layer="91"/>
+<wire x1="116.84" y1="162.56" x2="109.22" y2="162.56" width="0.1524" layer="91"/>
+<label x="109.22" y="162.56" size="1.778" layer="95"/>
+</segment>
+</net>

Commit message: Swapped power LED for right angle version
Parts:
- LED4: value (none) -> LED-902118128; device SparkFun:LED-3MM-NO_SILK -> morseSounder:LED-902118128
- R17, R18: value 10k -> 10K
- R3: value (none) -> 10K
Changed lines of the file:
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@@
 <part name="U$3" library="morseSounder" deviceset="P082D" device="TH"/>
 <part name="GND5" library="supply1" deviceset="GND" device=""/>
-<part name="R3" library="SparkFun" deviceset="RESISTOR" device="0805-RES"/>
+<part name="R3" library="SparkFun" deviceset="RESISTOR" device="0805-RES" value="10K"/>
 <part name="C4" library="SparkFun" deviceset="CAP" device="0805" value="100n"/>
 <part name="R4" library="SparkFun" deviceset="RESISTOR" device="0805-RES" value="10K"/>
@@
 <part name="GND26" library="supply1" deviceset="GND" device=""/>
 <part name="R30" library="SparkFun" deviceset="RESISTOR" device="0805-RES" value="22K"/>
-<part name="LED4" library="SparkFun" deviceset="LED" device="-3MM-NO_SILK"/>
+<part name="LED4" library="morseSounder" deviceset="LED-90" device="2118128"/>
 <part name="GND27" library="supply1" deviceset="GND" device=""/>
 <part name="R31" library="SparkFun" deviceset="RESISTOR" device="0805-RES" value="10"/>
@@
 <part name="Q4" library="SparkFun-DiscreteSemi" deviceset="MOSFET_PCH" device="-DMG2307L" value="2.5A/30V/105mΩ"/>
 <part name="P+7" library="supply1" deviceset="+12V" device=""/>
-<part name="R17" library="SparkFun" deviceset="RESISTOR" device="0805-RES" value="10k"/>
+<part name="R17" library="SparkFun" deviceset="RESISTOR" device="0805-RES" value="10K"/>
 <part name="Q5" library="transistor" deviceset="*-NPN-" device="SOT23-BEC" technology="MMBT3904LT1" value="MMBT3904"/>
-<part name="R18" library="SparkFun" deviceset="RESISTOR" device="0805-RES" value="10k"/>
+<part name="R18" library="SparkFun" deviceset="RESISTOR" device="0805-RES" value="10K"/>
 <part name="GND12" library="supply1" deviceset="GND" device=""/>
 <part name="TP9" library="SparkFun-Connectors" deviceset="TEST-POINT" device="3X5"/>
