File: PCB/morseSounder.brd (EAGLE design)
At the start: 56.6 x 82.7 mm, 84 parts, among them IC1 LM386M-1, IC5 LM321MF, J1 AVR_SPI_PRG_6PTH, J2 POWERPOLE_POWER25A_HORIZONTAL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, J3 POWER_JACKPTH, Q1 MMBT3904, Q2 MMBT3904, Q3 MMBT3904, Q4 2.5A/30V/105mΩ, Q5 MMBT3904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

Commit message: Swapped power LED for right angle version
Parts:
- LED4: value (none) -> LED-902118128; device SparkFun:LED3MM-NS -> morseSounder:MULTICOMP-2118128
- R17, R18: value 10k -> 10K
- R3: value (none) -> 10K
- moved R30 1.27 mm to (2.54, 10.2)
- moved LED4 0.29 mm to (3.81, 4.10)
Connections:
- net GND: now also LED4.P$2; no longer LED4.K
- net N$36: now also LED4.P$1; no longer LED4.A
Routing:
- net N$4: track 126.6 -> 127.9 mm
- net N$36: track 4.18 -> 5.16 mm
Other:
- board text added: "PWR"
- board text removed: "POWER"
Changed lines of the file:
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@@
 <setting verticaltext="up"/>
 </settings>
-<grid distance="0.05" unitdist="inch" unit="mm" style="lines" multiple="1" display="yes" altdistance="0.01" altunitdist="inch" altunit="mm"/>
+<grid distance="0.05" unitdist="inch" unit="mm" style="lines" multiple="1" display="yes" altdistance="0.003125" altunitdist="mic" altunit="mm"/>
 <layers>
 <layer number="1" name="Top" color="4" fill="1" visible="yes" active="yes"/>
@@
 <layer number="25" name="tNames" color="7" fill="1" visible="yes" active="yes"/>
 <layer number="26" name="bNames" color="7" fill="1" visible="yes" active="yes"/>
-<layer number="27" name="tValues" color="7" fill="1" visible="no" active="yes"/>
+<layer number="27" name="tValues" color="7" fill="1" visible="yes" active="yes"/>
 <layer number="28" name="bValues" color="7" fill="1" visible="no" active="yes"/>
-<layer number="29" name="tStop" color="7" fill="3" visible="yes" active="yes"/>
+<layer number="29" name="tStop" color="7" fill="3" visible="no" active="yes"/>
 <layer number="30" name="bStop" color="7" fill="6" visible="no" active="yes"/>
 <layer number="31" name="tCream" color="7" fill="4" visible="no" active="yes"/>
@@
 <wire x1="53.34" y1="30.48" x2="34.29" y2="30.48" width="0.4064" layer="25"/>
 <text x="49.53" y="14.224" size="1.27" layer="25" font="vector" ratio="10" rot="R90">Audio Amplifier</text>
-<text x="5.08" y="6.35" size="1.27" layer="25" font="vector" ratio="10" rot="R90">POWER</text>
+<text x="5.08" y="8.89" size="1.27" layer="25" font="vector" ratio="10" rot="R90">PWR</text>
 <text x="54.61" y="71.882" size="1.27" layer="25" font="vector" ratio="10" rot="R90">DC IN 12V</text>
 <text x="27.94" y="6.35" size="1.27" layer="25" font="vector" ratio="10" rot="R90" align="center">Tone
@@
 </element>
 <element name="U$3" library="morseSounder" package="P082D" value="P082DTH" x="34.29" y="0" locked="yes"/>
-<element name="R3" library="SparkFun" package="0805" value="" x="40.64" y="6.35" smashed="yes" rot="R180">
+<element name="R3" library="SparkFun" package="0805" value="10K" x="40.64" y="6.35" smashed="yes" rot="R180">
 <attribute name="NAME" x="42.164" y="6.35" size="0.6096" layer="25" font="vector"/>
 <attribute name="VALUE" x="41.656" y="7.747" size="0.4064" layer="27" rot="R180"/>
@@
 <attribute name="VALUE" x="46.99" y="82.55" size="0.4064" layer="27" rot="R180"/>
 </element>
-<element name="R30" library="SparkFun" package="0805" value="22K" x="2.54" y="8.89" smashed="yes" rot="R90">
-<attribute name="NAME" x="1.27" y="10.922" size="0.6096" layer="25" font="vector"/>
-<attribute name="VALUE" x="3.937" y="7.874" size="0.4064" layer="27" rot="R90"/>
-</element>
-<element name="LED4" library="SparkFun" package="LED3MM-NS" value="" x="3.81" y="3.81" smashed="yes">
-<attribute name="NAME" x="1.27" y="6.35" size="0.6096" layer="25" font="vector"/>
-<attribute name="VALUE" x="5.715" y="2.159" size="1.27" layer="27" ratio="10"/>
+<element name="R30" library="SparkFun" package="0805" value="22K" x="2.54" y="10.16" smashed="yes" rot="R90">
+<attribute name="NAME" x="1.27" y="12.192" size="0.6096" layer="25" font="vector"/>
+<attribute name="VALUE" x="3.937" y="9.144" size="0.4064" layer="27" rot="R90"/>
+</element>
+<element name="LED4" library="morseSounder" package="MULTICOMP-2118128" value="LED-902118128" x="3.81" y="4.1" smashed="yes">
+<attribute name="NAME" x="1.27" y="6.64" size="0.6096" layer="25" font="vector"/>
+<attribute name="VALUE" x="3.175" y="1.179" size="1.27" layer="27" ratio="10"/>
 </element>
 <element name="R31" library="SparkFun" package="0805" value="10" x="44.45" y="57.15" smashed="yes">
@@
 <attribute name="VALUE" x="29.591" y="41.91" size="0.6096" layer="27" font="vector" ratio="20" rot="R90" align="top-center"/>
 </element>
-<element name="R17" library="SparkFun" package="0805" value="10k" x="27.94" y="38.1" smashed="yes">
+<element name="R17" library="SparkFun" package="0805" value="10K" x="27.94" y="38.1" smashed="yes">
 <attribute name="NAME" x="29.718" y="38.1" size="0.6096" layer="25" font="vector"/>
 <attribute name="VALUE" x="26.924" y="36.703" size="0.4064" layer="27"/>
@@
 <attribute name="VALUE" x="26.035" y="31.115" size="1.27" layer="27"/>
 </element>
-<element name="R18" library="SparkFun" package="0805" value="10k" x="22.86" y="34.29" smashed="yes" rot="R270">
+<element name="R18" library="SparkFun" package="0805" value="10K" x="22.86" y="34.29" smashed="yes" rot="R270">
 <attribute name="NAME" x="21.844" y="33.528" size="0.6096" layer="25" font="vector" rot="R90"/>
 <attribute name="VALUE" x="21.463" y="35.306" size="0.4064" layer="27" rot="R270"/>
@@
 <contactref element="S1" pad="3"/>
 <contactref element="J2" pad="BLACK"/>
-<contactref element="LED4" pad="K"/>
+<contactref element="LED4" pad="P$2"/>
 <contactref element="U$5" pad="3"/>
 <contactref element="C17" pad="1"/>
@@
 <signal name="N$36">
 <contactref element="R30" pad="1"/>
-<contactref element="LED4" pad="A"/>
-<wire x1="2.54" y1="7.99" x2="2.54" y2="3.81" width="1" layer="1"/>
+<contactref element="LED4" pad="P$1"/>
+<wire x1="2.54" y1="9.26" x2="2.54" y2="4.1" width="1" layer="1"/>
 </signal>
 <signal name="N$2">
@@
 <wire x1="52.07" y1="1.27" x2="11.43" y2="1.27" width="0.4064" layer="1"/>
 <wire x1="11.43" y1="1.27" x2="6.35" y2="6.35" width="0.4064" layer="1"/>
-<wire x1="6.35" y1="6.35" x2="6.35" y2="7.62" width="0.4064" layer="1"/>
-<wire x1="6.35" y1="7.62" x2="4.18" y2="9.79" width="0.4064" layer="1"/>
-<wire x1="2.54" y1="9.79" x2="4.18" y2="9.79" width="0.4064" layer="1"/>
+<wire x1="6.35" y1="6.35" x2="6.35" y2="8.89" width="0.4064" layer="1"/>
+<wire x1="6.35" y1="8.89" x2="4.18" y2="11.06" width="0.4064" layer="1"/>
+<wire x1="2.54" y1="11.06" x2="4.18" y2="11.06" width="0.4064" layer="1"/>
 <contactref element="D4" pad="C"/>
 <wire x1="45.35" y1="57.15" x2="45.35" y2="58.79" width="0.4064" layer="1"/>
